File: boards/v3.1/board.kicad_sch (KiCad schematic)
At the start: 51 parts, among them J1 KF301-2P, J2 KF301-2P, J3 KF301-2P, J4 KF301-2P, J5 KF301-2P, J6 KF301-2P, P1 Pin Header, P2 Pin Header, P3 Pin Header, P4 Pin Header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

Commit message: Update the list of components and calcs
Other:
- title: Energy Guardian V3.1 Schematic -> Power Vision V3.1 Schematic
Changed lines of the file:
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@@
   (paper "A4")
   (title_block
-    (title "Energy Guardian V3.1 Schematic")
+    (title "Power Vision V3.1 Schematic")
     (date "12/05/2024")
     (rev "1.1")
