File: boards/v3.2/board.kicad_sch (KiCad schematic)
At the start: 51 parts, among them J1 KF301-2P, J2 KF301-2P, J3 KF301-2P, J4 KF301-2P, J5 KF301-2P, J6 KF301-2P, P1 Pin Header, P2 Pin Header, P3 Pin Header, P4 Pin Header, P5 Pin Header, SW1 SS-12D00G 4mm, SW2 SS-12D00G 4mm, T1 ZMPT101B, T2 ZMPT101B, T3 ZMPT101B

Commit message: update all parts of project
Parts:
- removed SW1, SW2: SS-12D00G 4mm, Connector_PinHeader_2.54mm:PinHeader_1x03_P2.54mm_Vertical, symbol Switch:SW_DPDT_x2
- added SW1: SS-12D00G 4mm, Connector_PinHeader_2.54mm:PinHeader_1x03_P2.54mm_Vertical, symbol Switch:SW_Nidec_CAS-120A1
- C1: value 16V 1000µF -> 35V 47µF; footprint Capacitor_THT:CP_Radial_D6.3mm_P2.50mm -> Capacitor_THT:CP_Radial_Tantal_D6.0mm_P2.50mm
- C2: footprint Capacitor_THT:CP_Radial_D5.0mm_P2.00mm -> Capacitor_THT:CP_Radial_Tantal_D5.0mm_P2.50mm
- PS1: value HLK-5M05 -> HLK-10M24
- renumbered T1 to TP1, T2 to TP2, T3 to TP3
Connections:
- net Current A: now also AMP2.7, MCU1.J1_6 (GPIO6), R9.1; no longer AMP3.1, AMP3.2 (-), MCU1.J1_7 (GPIO7)
- net Current B: now also MCU1.J1_12 (GPIO8), R10.1; no longer AMP3.6 (-), MCU1.J1_6 (GPIO6)
- net Current C: now also MCU1.J1_16 (GPIO10), R11.1; no longer AMP4.2 (-), MCU1.J1_5 (GPIO5)
- net Current N: now also MCU1.J1_15 (GPIO9), R12.1; no longer AMP4.6 (-), MCU1.J1_4 (GPIO4)
- net GND: no longer MCU1.J1_22 (GND), MCU1.J3_22 (GND__3)
- net TC A-1: now also AMP1.3 (+), AMP1.6 (-), AMP1.7, AMP2.3 (+), AMP2.5 (+), AMP3.5 (+), AMP4.3 (+), AMP4.5 (+), J3.1 (Pin_1), J4.1 (Pin_1), J5.1 (Pin_1), J6.1 (Pin_1), P2.1 (Pin_1), TP1.4, TP2.4, TP3.4; no longer J3.2 (Pin_2), R9.1
- net TC A-2: now also AMP2.6 (-), J3.2 (Pin_2); no longer AMP1.1, AMP1.2 (-), J3.1 (Pin_1), J4.1 (Pin_1), J5.1 (Pin_1), J6.1 (Pin_1), P2.1 (Pin_1), R10.2, R11.2, R12.2, R6.2, R7.2, R8.2, TP1.4, TP2.4, TP3.4
- net V1.65: now also AMP1.5 (+); no longer AMP1.3 (+)
- net Vin: now also C1.1, SW1.1 (C)
- net Wave A: now also AMP1.1, DZ1.2 (A), DZ2.1 (K), MCU1.J1_4 (GPIO4), P4.1 (Pin_1), R6.2; no longer AMP2.5 (+), R6.1, TP1.3
- net Wave B: now also AMP2.1, DZ3.2 (A), DZ4.1 (K), MCU1.J1_5 (GPIO5), P4.2 (Pin_2), R7.2; no longer AMP2.3 (+), R7.1, TP2.3
- net Wave C: now also AMP3.1, DZ5.2 (A), DZ6.1 (K), MCU1.J1_7 (GPIO7), P4.3 (Pin_3), R8.2; no longer AMP1.5 (+), R8.1, TP3.3
- net Power: no longer names the net of PS1.4 (+Vout)
- net Power: now also SW1.2 (B); no longer C1.1
- net System Type: no longer names the net of MCU1.J3_4 (GPIO1)
- removed net TC B-1: AMP3.5 (+), J4.2 (Pin_2), R10.1
- removed net TC C-1: AMP4.3 (+), J5.2 (Pin_2), R11.1
- removed net TC N-1: AMP4.5 (+), J6.2 (Pin_2), R12.1
- removed net Treated Wave A: AMP2.6 (-), AMP2.7, DZ5.2 (A), DZ6.1 (K), MCU1.J1_12 (GPIO8), P4.1 (Pin_1)
- removed net Treated Wave B: AMP2.1, AMP2.2 (-), DZ3.2 (A), DZ4.1 (K), MCU1.J1_15 (GPIO9), P4.2 (Pin_2)
- removed net Treated Wave C: AMP1.6 (-), AMP1.7, DZ1.2 (A), DZ2.1 (K), MCU1.J1_16 (GPIO10), P4.3 (Pin_3)
- new net TC B-2: AMP3.6 (-), J4.2 (Pin_2), R10.2
- new net TC C-2: AMP4.2 (-), J5.2 (Pin_2), R11.2
- new net TC N-2: AMP4.6 (-), J6.2 (Pin_2), R12.2
- new net TP A-1: AMP1.2 (-), R6.1, TP1.3
- new net TP B-1: AMP2.2 (-), R7.1, TP2.3
- new net TP C-1: AMP3.2 (-), R8.1, TP3.3
Other:
- note added: "After selecting the ideal resistor for your application, according to the tables, remember to modify the value of the variables "CURRENT TYPE", "VOLTAGE_TYPE" and "SYSTEM_TYPE" in the MCU code according to what's in the tables"
- note added: "Biphasic (2P)"
- note added: "Biphasic (2P+N)"
- note added: "Single-phase (P+N)"
- note added: "System Type"
- note added: "Three-phase (3P+N)"
- note added: "Type"
- note added: "Type of Electrical System"
- note removed: "Switch System Type"
- note removed: "Then select the ideal resistor for your application, according to the tables, so remember to modify the value of the variables "CURRENT_TYPE" and "VOLTAGE_TYPE" in the MCU code according to what is in the table!"
- title: Energy Guardian V3.1 Schematic -> Energy Guardian V3.2 Schematic
- moved on the sheet: AMP1C, AMP2A, AMP2C, AMP3B, AMP3C, AMP4A, AMP4B, AMP4C, C2, DZ1, DZ10, DZ11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
