File: boards/v3.2/board.kicad_pcb (KiCad board)
At the start: 2 copper layers, 94.5 x 92.7 mm, 51 parts, among them J1 KF301-2P, J2 KF301-2P, J3 KF301-2P, J4 KF301-2P, J5 KF301-2P, J6 KF301-2P, P1 Pin Header, P2 Pin Header, P3 Pin Header, P4 Pin Header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

Commit message: The last board and documentation update
Connections:
- DZ1 pad 1: GND -> Vcc
- DZ10 pad 2: Vcc -> GND
- DZ11 pad 1: GND -> Vcc
- DZ12 pad 2: Vcc -> GND
- DZ13 pad 1: GND -> Vcc
- DZ14 pad 2: Vcc -> GND
- DZ2 pad 2: Vcc -> GND
- DZ3 pad 1: GND -> Vcc
- DZ4 pad 2: Vcc -> GND
- DZ5 pad 1: GND -> Vcc
- DZ6 pad 2: Vcc -> GND
- DZ7 pad 1: GND -> Vcc
- DZ8 pad 2: Vcc -> GND
- DZ9 pad 1: GND -> Vcc
Routing:
- net GND: track 200.9 -> 255.6 mm
- net Vcc: track 65.8 -> 113.1 mm
