File: boards/v4.0/board.kicad_pcb (KiCad board)
At the start: 2 copper layers, 75.4 x 74.9 mm, 63 parts, among them J1 KF301-2P, J2 KF301-2P, J3 KF301-2P, J4 KF301-2P, J5 KF301-2P, J6 KF301-2P, J7 KF301-2P, P1 Pin Header, P2 Pin Header, P3 Pin Header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

Commit message: Board IDs Correction and update documentation
Parts:
- moved AMP2 8.68 mm to (134.8, 84.4)
- moved DZ14 8.68 mm to (168.2, 86.0)
- moved DZ4 8.68 mm to (168.2, 78.8)
- moved DZ5 8.68 mm to (176.0, 82.4)
- moved DZ6 8.68 mm to (168.2, 82.4)
- moved J1 8.68 mm to (112.7, 49.9)
- moved P1 8.68 mm to (143.4, 69.2)
- moved P3 8.68 mm to (166.5, 70.1)
- moved R13 8.68 mm to (134.8, 71.5)
- moved R15 8.68 mm to (134.8, 106.4)
- moved R16 8.68 mm to (145.2, 100.3)
- moved R17 8.68 mm to (155.3, 100.3)
- moved R18 8.68 mm to (165.5, 100.3)
- moved R6 8.68 mm to (134.8, 62.6)
- moved R7 8.68 mm to (134.8, 80.0)
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- renumbered PS2 to PS1

Commit message: Initial tests of microcontroller code
Parts:
- added R20: 50Ω, Resistor_SMD:R_1210_3225Metric, F.Cu at (146.6, 61.8)
Connections:
- AMP8 pad 1: TC A-1 -> Net-(AMP8A--)
- AMP8 pad 2: TC A-1 -> Net-(AMP8A--)
Routing:
- net Net-(AMP8A--): track 0.00 -> 20.5 mm, vias 0 -> 2
- net TC A-1: track 244.1 -> 235.8 mm, vias 13 -> 12

Commit message: Code update
Parts:
- R6, R7, R8: value RSvolt -> 430Ω
Changed lines of the file:
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@@
         (effects (font (size 1 1) (thickness 0.15)))
     )
-    (fp_text value "RSvolt" (at 0 2.28) (layer "F.Fab") hide
+    (fp_text value "430Ω" (at 0 2.28) (layer "F.Fab") hide
         (effects (font (size 1 1) (thickness 0.15)))
     )
@@
         (effects (font (size 1 1) (thickness 0.15)))
     )
-    (fp_text value "RSvolt" (at 0 2.28) (layer "F.Fab") hide
+    (fp_text value "430Ω" (at 0 2.28) (layer "F.Fab") hide
         (effects (font (size 1 1) (thickness 0.15)))
     )
-    (fp_text user "${VALUE}" (at 0 0 90) (layer "F.SilkS")
+    (fp_text user "${REFERENCE}" (at 0 0 90) (layer "F.SilkS")
         (effects (font (size 0.4 0.4) (thickness 0.1)))
     )
@@
         (effects (font (size 1 1) (thickness 0.15)))
     )
-    (fp_text value "RSvolt" (at 0 2.28) (layer "F.Fab") hide
+    (fp_text value "430Ω" (at 0 2.28) (layer "F.Fab") hide
         (effects (font (size 1 1) (thickness 0.15)))
     )
@@
     (fp_line (start 1.6 1.245) (end -1.6 1.245)
       (stroke (width 0.1) (type solid)) (layer "F.Fab"))
-    (pad "1" smd roundrect (at -1.4625 0 90) (size 1.125 2.65) (layers "F.Cu" "F.Paste" "F.Mask") (roundrect_rratio 0.222222)
+    (pad "1" smd roundrect (at -1.4625 0 90) (size 1.125 2.65) (layers "F.Cu" "F.Paste" "F.Mask") (roundrect_rratio 0.2222222222)
       (net 15 "TC A-1") (pintype "passive"))
-    (pad "2" smd roundrect (at 1.4625 0 90) (size 1.125 2.65) (layers "F.Cu" "F.Paste" "F.Mask") (roundrect_rratio 0.222222)
+    (pad "2" smd roundrect (at 1.4625 0 90) (size 1.125 2.65) (layers "F.Cu" "F.Paste" "F.Mask") (roundrect_rratio 0.2222222222)
       (net 80 "Net-(AMP8A--)") (pintype "passive"))
     (model "${KICAD6_3DMODEL_DIR}/Resistor_SMD.3dshapes/R_1210_3225Metric.wrl"
@@
   (via (at 154.5596 71.3486) (size 0.6) (drill 0.4) (layers "F.Cu" "B.Cu") (free) (net 27))
   (segment (start 154.5596 62.0776) (end 154.5596 71.3486) (width 0.2) (layer "B.Cu") (net 27))
-  (segment (start 156.9476 62.3566) (end 156.9476 59.6646) (width 0.2) (layer "F.Cu") (net 28))
-  (segment (start 156.3376 62.9666) (end 156.9476 62.3566) (width 0.2) (layer "F.Cu") (net 28))
   (segment (start 153.2896 72.7526) (end 153.2766 72.7656) (width 0.2) (layer "F.Cu") (net 28))
+  (segment (start 156.9476 62.3566) (end 156.9476 59.6646) (width 0.2) (layer "F.Cu") (net 28))
   (segment (start 153.2896 62.9666) (end 156.3376 62.9666) (width 0.2) (layer "F.Cu") (net 28))
+  (segment (start 156.3376 62.9666) (end 156.9476 62.3566) (width 0.2) (layer "F.Cu") (net 28))
   (segment (start 153.2896 71.3486) (end 153.2896 72.7526) (width 0.2) (layer "F.Cu") (net 28))
   (via (at 153.2896 71.3486) (size 0.6) (drill 0.4) (layers "F.Cu" "B.Cu") (free) (net 28))
