File: boards/v5.0/board.kicad_pcb (KiCad board)
At the start: 2 copper layers, 120 x 86 mm, 81 parts, among them J1 KF301-2P, J2 KF301-2P, J3 KF301-2P, J4 KF301-2P, J5 KF301-2P, J6 KF301-2P, J7 KF301-2P, P1 Pin Header, P2 Pin Header, P3 Pin Header, P4 Pin Header, P5 Conn_01x07, P6 Pin Header, SW1 SS-12D00G 4mm, U2 LD1086#50

Commit message: Update board v5.0 docs
Parts:
- removed AMP10, AMP11, AMP12, AMP13, AMP14, AMP15, AMP16, AMP9: TL082, Package_SO:SO-8_3.9x4.9mm_P1.27mm
- removed C17, C18: 16V 1uF, Capacitor_SMD:C_0402_1005Metric
- removed J7: KF301-2P, TerminalBlock:TerminalBlock_bornier-2_P5.08mm
- removed MCU1: ESP32-S3-WROOM-1-N16R8, SnapEDA Library:XCVR_ESP32-S3-WROOM-2-N32R8V
- removed R30, R31, R32: 50Ω, Resistor_SMD:R_1206_3216Metric
- removed R33, R34, R35: 50Ω, Resistor_SMD:R_1210_3225Metric
- added C10: 10V 0.1uF, Capacitor_SMD:C_0603_1608Metric, F.Cu at (36.0, 86.4)
- added C3: 10V 47µF, Capacitor_Tantalum_SMD:CP_EIA-7343-31_Kemet-D, F.Cu at (21.7, 77.7)
- added C4: 10V 0.1µF, Capacitor_SMD:C_0603_1608Metric, F.Cu at (38.4, 63.6)
- added C5: 10V 0.1µF, Capacitor_SMD:C_0603_1608Metric, F.Cu at (38.4, 66.2)
- added C6: 10V 0.1µF, Capacitor_SMD:C_0603_1608Metric, F.Cu at (38.4, 68.7)
- added C7: 10V 0.1µF, Capacitor_SMD:C_0603_1608Metric, F.Cu at (44.5, 63.6)
- added C8: 10V 0.1µF, Capacitor_SMD:C_0603_1608Metric, F.Cu at (44.5, 66.2)
- added C9: 10V 0.1uF, Capacitor_SMD:C_0603_1608Metric, F.Cu at (36.0, 83.8)
- added D1: 1N4007, Diode_THT:D_DO-41_SOD81_P10.16mm_Horizontal, F.Cu at (14.4, 84.7)
- added P7: Pin Header, Connector_PinHeader_2.54mm:PinHeader_1x03_P2.54mm_Vertical, F.Cu at (47.0, 84.9)
- added P8: Pin Header, Connector_PinHeader_2.54mm:PinHeader_1x04_P2.54mm_Vertical, F.Cu at (42.4, 84.9)
- added Q1: FZT948TA, Package_TO_SOT_SMD:SOT-223, F.Cu at (11.8, 66.5)
- added Q2: FZT948TA, Package_TO_SOT_SMD:SOT-223, F.Cu at (11.8, 74.8)
- added R10: RVolt, Resistor_SMD:R_1206_3216Metric, F.Cu at (9.69, 94.1)
- added R11: RVolt, Resistor_SMD:R_1206_3216Metric, F.Cu at (9.69, 97.4)
- added R12: RVolt, Resistor_SMD:R_1206_3216Metric, F.Cu at (9.69, 100.7)
- added R13: 10kΩ, Resistor_SMD:R_1206_3216Metric, F.Cu at (31.2, 84.2)
- added R14: 10kΩ, Resistor_SMD:R_1206_3216Metric, F.Cu at (31.2, 87.5)
- added R15: 50Ω, Resistor_SMD:R_1206_3216Metric, F.Cu at (31.2, 90.8)
- added R16: 430Ω, Resistor_SMD:R_1206_3216Metric, F.Cu at (31.2, 94.1)
- added R17: 50Ω, Resistor_SMD:R_1206_3216Metric, F.Cu at (31.2, 97.4)
- added R3: 1kΩ, Resistor_SMD:R_0603_1608Metric, F.Cu at (38.4, 71.2)
- added R4: 1kΩ, Resistor_SMD:R_0603_1608Metric, F.Cu at (38.4, 73.7)
- added R5: 1kΩ, Resistor_SMD:R_0603_1608Metric, F.Cu at (38.4, 76.2)
- added R6: 1kΩ, Resistor_SMD:R_0603_1608Metric, F.Cu at (38.4, 78.7)
- added R7: 10kΩ, Resistor_SMD:R_1206_3216Metric, F.Cu at (9.69, 84.2)
- added R8: 1MΩ, Resistor_SMD:R_1206_3216Metric, F.Cu at (9.69, 87.5)
- added R9: 1MΩ, Resistor_SMD:R_1206_3216Metric, F.Cu at (9.69, 90.8)
- added U1: LD1086#50, Package_TO_SOT_SMD:TO-263-3_TabPin2, F.Cu at (27.5, 68.6)
- added U3: PC817, Package_DIP:DIP-4_W7.62mm, F.Cu at (14.1, 88.9)
- C1: value 50V 100µF -> 100V 0.1µF; footprint Capacitor_SMD:CP_Elec_10x10 -> Capacitor_SMD:C_1206_3216Metric
- C11, C12, C13, C14, C15, C16: value 16V 1uF -> 10V 0.1uF; footprint Capacitor_SMD:C_0402_1005Metric -> Capacitor_SMD:C_0603_1608Metric
- C2: value 10V 47µF -> 50V 100µF; footprint Capacitor_Tantalum_SMD:CP_EIA-7343-31_Kemet-D -> Capacitor_SMD:CP_Elec_10x10
- J1, J3, J4, J5, J6: value KF301-2P -> Screw_Terminal_01x02; footprint TerminalBlock:TerminalBlock_bornier-2_P5.08mm -> TerminalBlock_Phoenix:TerminalBlock_Phoenix_MKDS-1,5-2-5.08_1x02_P5.08mm_Horizontal
- J2: value KF301-2P -> Screw_Terminal_01x04; footprint TerminalBlock:TerminalBlock_bornier-2_P5.08mm -> TerminalBlock_Phoenix:TerminalBlock_Phoenix_MKDS-1,5-4-5.08_1x04_P5.08mm_Horizontal
- P1: value Pin Header -> Pin Socket 2.54mm 02x22; footprint Connector_PinHeader_2.54mm:PinHeader_1x03_P2.54mm_Vertical -> Connector_PinSocket_2.54mm:PinSocket_2x22_P2.54mm_Vertical
- P2: value Pin Header -> Pin Socket 2.54mm 01x22; footprint Connector_PinHeader_2.54mm:PinHeader_1x01_P2.54mm_Vertical -> Connector_PinSocket_2.54mm:PinSocket_1x22_P2.54mm_Vertical
- P3: value Pin Header -> Pin Socket 2.54mm 2x20; footprint Connector_PinHeader_2.54mm:PinHeader_1x03_P2.54mm_Vertical -> Connector_PinSocket_2.54mm:PinSocket_2x20_P2.54mm_Vertical
- P4: footprint Connector_PinHeader_2.54mm:PinHeader_1x04_P2.54mm_Vertical -> Connector_PinHeader_2.54mm:PinHeader_1x03_P2.54mm_Vertical
- P5: value Conn_01x07 -> Pin Header; footprint Connector_PinHeader_2.54mm:PinHeader_1x07_P2.54mm_Vertical -> Connector_PinHeader_2.54mm:PinHeader_1x04_P2.54mm_Vertical
- P6: value Pin Header -> Conn_01x07; footprint Connector_PinHeader_2.54mm:PinHeader_1x04_P2.54mm_Vertical -> Connector_PinHeader_2.54mm:PinHeader_1x07_P2.54mm_Vertical
- R1: value 10kΩ -> 2Ω; footprint Resistor_SMD:R_1206_3216Metric -> Resistor_SMD:R_0603_1608Metric
- R18, R20: value RVolt -> 430Ω
- R19: value RVolt -> 50Ω
- R2: value 10kΩ -> 0.2Ω; footprint Resistor_SMD:R_1206_3216Metric -> Resistor_SMD:R_2512_6332Metric
- R21, R23: value 430Ω -> 50Ω
- R22: value 430Ω -> Rcurr
- R24, R29: footprint Resistor_SMD:R_1206_3216Metric -> Resistor_SMD:R_1210_3225Metric
- R25, R27: value Rcurr -> 50Ω
- R28: value 50Ω -> Rcurr; footprint Resistor_SMD:R_1206_3216Metric -> Resistor_SMD:R_1210_3225Metric
- U2: value LD1086#50 -> TXS0108EPW; footprint Package_TO_SOT_SMD:TO-263-3_TabPin2 -> Package_SO:TSSOP-20_4.4x6.5mm_P0.65mm
- moved P2 78.3 mm to (-96.5, 96.0)
- moved P1 74.2 mm to (-96.5, 100.0)
- moved P3 57.7 mm to (-91.4, 86.4)
Connections:
- AMP1 pad 2: /Signals Conditioning/PT A-2 -> /Signals Acquisition/PT A-2
- AMP1 pad 3: Vref -> /Signals Acquisition/PT A-1
- AMP1 pad 8: Vin -> /Microcomputer/5V
- AMP2 pad 2: /Signals Conditioning/PT B-2 -> /Signals Acquisition/PT B-2
- AMP2 pad 3: Vref -> /Signals Acquisition/PT A-1
- AMP2 pad 8: Vin -> /Microcomputer/5V
- AMP3 pad 2: /Signals Conditioning/PT C-2 -> /Signals Acquisition/PT C-2
- AMP3 pad 3: Vref -> /Signals Acquisition/PT A-1
- AMP3 pad 8: Vin -> /Microcomputer/5V
- AMP4 pad 3: Vref -> /Signals Acquisition/PT A-1
- AMP4 pad 8: Vin -> /Microcomputer/5V
- AMP5 pad 3: Vref -> /Signals Acquisition/PT A-1
- AMP5 pad 8: Vin -> /Microcomputer/5V
- AMP6 pad 3: Vref -> /Signals Acquisition/PT A-1
- AMP6 pad 8: Vin -> /Microcomputer/5V
- AMP7 pad 3: Vref -> /Signals Acquisition/PT A-1
- AMP7 pad 8: Vin -> /Microcomputer/5V
- AMP8 pad 8: Vin -> /Microcomputer/5V
- C1 pad 1: Vin -> /Power/IN+
- C11 pad 1: Vref -> Net-(AMP2B-+)
- C12 pad 1: Net-(AMP1B-+) -> Net-(AMP3B-+)
- C13 pad 1: Net-(AMP2B-+) -> Net-(AMP4B-+)
- C14 pad 1: Net-(AMP3B-+) -> Net-(AMP5B-+)
- C15 pad 1: Net-(AMP4B-+) -> Net-(AMP6B-+)
- C16 pad 1: Net-(AMP5B-+) -> Net-(AMP7B-+)
- C2 pad 1: Vcc -> Net-(Q1-C)
- DZ1 pad 1: Wave A -> /Microcontroller/ADC1_0
- DZ10 pad 1: Current B -> /Microcontroller/ADC1_5
- DZ11 pad 1: Vcc -> /Microcomputer/3.3V
- DZ11 pad 2: Current C -> /Microcontroller/ADC1_4
- DZ12 pad 1: Current C -> /Microcontroller/ADC1_4
- DZ13 pad 1: Vcc -> /Microcomputer/3.3V
- DZ13 pad 2: Current N -> /Microcontroller/ADC1_6
- DZ14 pad 1: Current N -> /Microcontroller/ADC1_6
- DZ2 pad 1: Vcc -> /Microcomputer/3.3V
- DZ2 pad 2: Wave A -> /Microcontroller/ADC1_0
- DZ3 pad 1: Wave B -> /Microcomputer/3.3V
- DZ3 pad 2: Earth -> /Microcontroller/ADC1_1
- DZ4 pad 1: Vcc -> /Microcontroller/ADC1_1
- DZ4 pad 2: Wave B -> Earth
- DZ5 pad 1: Wave C -> /Microcomputer/3.3V
- DZ5 pad 2: Earth -> /Microcontroller/ADC1_2
- DZ6 pad 1: Vcc -> /Microcontroller/ADC1_2
- DZ6 pad 2: Wave C -> Earth
- DZ7 pad 1: Vcc -> /Microcomputer/3.3V
- DZ7 pad 2: Current A -> /Microcontroller/ADC1_3
- DZ8 pad 1: Current A -> /Microcontroller/ADC1_3
- DZ9 pad 1: Vcc -> /Microcomputer/3.3V
- DZ9 pad 2: Current B -> /Microcontroller/ADC1_5
- J1 pad 1: 5V-27V -> Earth
- J1 pad 2: Earth -> /Power/IN+
- J2 pad 1: Line A -> /Signals Acquisition/Neutral
- J2 pad 2: Line B -> /Signals Acquisition/Line C
- J3 pad 1: Line C -> /Signals Acquisition/PT A-1
- J3 pad 2: Neutral -> /Signals Conditioning/CT A-2
- J4 pad 1: TC A-1 -> /Signals Conditioning/CT B-2
- J4 pad 2: TC A-2 -> /Signals Acquisition/PT A-1
- J5 pad 1: TC B-1 -> /Signals Conditioning/CT C-2
- J5 pad 2: TC B-2 -> /Signals Acquisition/PT A-1
- J6 pad 1: TC C-1 -> /Signals Conditioning/CT N-2
- J6 pad 2: TC C-2 -> /Signals Acquisition/PT A-1
- P1 pad 1: Earth -> /Microcomputer/5V
- P1 pad 2: UART TX -> /Microcomputer/5V
- P1 pad 3: UART RX -> /Microcontroller/RESET
- P2 pad 1: Vref -> unconnected-(P2-Pin_1-Pad1)
- P3 pad 1: Wave A -> /Microcomputer/5V
- P3 pad 2: Wave B -> /Microcomputer/I2C SDA
- P3 pad 3: Wave C -> /Microcomputer/I2C SCL
- P4 pad 1: Current A -> /Microcomputer/TX_0
- P4 pad 2: Current B -> /Microcomputer/RX_0
- P4 pad 3: Current C -> Earth
- P5 pad 1: Earth -> /Microcomputer/I2C SDA
- P5 pad 2: Vcc -> /Microcomputer/I2C SCL
- P5 pad 3: SPI MOSI -> /Microcomputer/5V
- P5 pad 4: SPI MISO -> Earth
- P6 pad 1: Earth -> /Microcontroller/SPI_DC
- P6 pad 2: Vcc -> /Microcontroller/SPI_CS
- P6 pad 3: I2C SDA -> /Microcontroller/SPI_SCK
- P6 pad 4: I2C SCL -> /Microcontroller/SPI_MISO
- R1 pad 1: /Signals Conditioning/3.3V -> Net-(Q1-E)
- R1 pad 2: Net-(AMP8A-+) -> Net-(Q1-C)
- R18 pad 1: Net-(R18-Pad1) -> /Signals Acquisition/PT B-2
- R18 pad 2: Line A -> Net-(AMP2B-+)
- R19 pad 1: Net-(R19-Pad1) -> Net-(AMP2B--)
- R19 pad 2: Line B -> /Microcontroller/ADC1_1
- R2 pad 1: Earth -> Net-(Q1-E)
- R2 pad 2: Net-(AMP8A-+) -> Net-(Q1-B)
- R20 pad 1: Net-(R20-Pad1) -> /Signals Acquisition/PT C-2
- R20 pad 2: Line C -> Net-(AMP3B-+)
- R21 pad 1: /Signals Conditioning/PT A-2 -> Net-(AMP3B--)
- R21 pad 2: Net-(AMP1B-+) -> /Microcontroller/ADC1_2
- R22 pad 1: /Signals Conditioning/PT B-2 -> Net-(AMP4B-+)
- R22 pad 2: Net-(AMP2B-+) -> /Signals Conditioning/CT A-2
- R23 pad 1: /Signals Conditioning/PT C-2 -> Net-(AMP4B--)
- R23 pad 2: Net-(AMP3B-+) -> /Microcontroller/ADC1_3
- R24 pad 1: Net-(AMP4B-+) -> Net-(AMP5B-+)
- R24 pad 2: /Signals Conditioning/CT A-2 -> /Signals Conditioning/CT B-2
- R25 pad 1: Net-(AMP5B-+) -> Net-(AMP5B--)
- R25 pad 2: /Signals Conditioning/CT B-2 -> /Microcontroller/ADC1_5
- R27 pad 1: Net-(AMP7B-+) -> Net-(AMP6B--)
- R27 pad 2: /Signals Conditioning/CT N-2 -> /Microcontroller/ADC1_4
- R28 pad 1: Vref -> Net-(AMP7B-+)
- R28 pad 2: Net-(AMP8A--) -> /Signals Conditioning/CT N-2
- R29 pad 1: Net-(AMP1B--) -> Net-(AMP7B--)
- R29 pad 2: /Signals Conditioning/Wave A -> /Microcontroller/ADC1_6
- SW1 pad 1: 5V-30V -> /Power/IN+
- SW1 pad 2: Vin -> Net-(Q1-E)
- TP1 pad 1: Net-(R18-Pad1) -> Net-(R10-Pad1)
- TP1 pad 2: Neutral -> /Signals Acquisition/Neutral
- TP1 pad 3: TP A-1 -> /Signals Acquisition/PT A-1
- TP1 pad 4: TP A-2 -> /Signals Acquisition/PT A-2
- TP2 pad 1: Net-(R19-Pad1) -> Net-(R11-Pad1)
- TP2 pad 2: Neutral -> /Signals Acquisition/Neutral
- TP2 pad 3: TP B-1 -> /Signals Acquisition/PT A-1
- TP2 pad 4: TP B-2 -> /Signals Acquisition/PT B-2
- TP3 pad 1: Net-(R20-Pad1) -> Net-(R12-Pad1)
- TP3 pad 2: Neutral -> /Signals Acquisition/Neutral
- TP3 pad 3: TP C-1 -> /Signals Acquisition/PT A-1
- TP3 pad 4: TP C-2 -> /Signals Acquisition/PT C-2
- U2 pad 1: Earth -> /Microcomputer/RX_4
- U2 pad 2: Vcc -> /Microcomputer/3.3V
- U2 pad 3: Vin -> /Microcomputer/TX_4
Routing:
- net (no net): track 24.3 -> 427.3 mm, vias 0 -> 5
- net TC A-1: track 249.2 -> 0.00 mm, vias 13 -> 0
- net Vref: track 0.00 -> 206.7 mm
- net Vcc: track 140.4 -> 0.00 mm, vias 11 -> 0
- net Vin: track 122.5 -> 0.00 mm, vias 9 -> 0
- net Wave B: track 86.4 -> 0.00 mm, vias 3 -> 0
- net Current A: track 77.1 -> 0.00 mm, vias 5 -> 0
- net Current N: track 71.5 -> 0.00 mm, vias 4 -> 0
- net /Microcontroller/ADC1_6: track 0.00 -> 71.5 mm, vias 0 -> 4
- net /Microcontroller/ADC1_3: track 0.00 -> 63.7 mm, vias 0 -> 1
- net Current C: track 60.1 -> 0.00 mm, vias 4 -> 0
- net /Microcontroller/ADC1_4: track 0.00 -> 60.1 mm
- net Current B: track 56.9 -> 0.00 mm, vias 4 -> 0
- net /Microcontroller/ADC1_5: track 0.00 -> 56.9 mm, vias 0 -> 1
- net Neutral: track 52.0 -> 0.00 mm
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
Commit message: Update in the V5 board
Parts:
- added P10: Pin Header, Connector_PinHeader_2.54mm:PinHeader_1x03_P2.54mm_Vertical, F.Cu at (111.0, 53.0)
- added P9: Pin Header, Connector_PinHeader_2.54mm:PinHeader_1x03_P2.54mm_Vertical, F.Cu at (56.9, 95.8)
- P3: value Pin Socket 2.54mm 2x20 -> Conn_01x20; footprint Connector_PinSocket_2.54mm:PinSocket_2x20_P2.54mm_Vertical -> Connector_PinHeader_2.54mm:PinHeader_1x20_P2.54mm_Vertical
- P4: value Pin Header -> Conn_01x20; footprint Connector_PinHeader_2.54mm:PinHeader_1x03_P2.54mm_Vertical -> Connector_PinHeader_2.54mm:PinHeader_1x20_P2.54mm_Vertical
- moved TP1 253.9 mm to (112.5, 108.1), turned to 90 degrees
- moved TP2 240.9 mm to (95.1, 108.1), turned to 90 degrees
- moved TP3 229.9 mm to (77.7, 108.1), turned to 90 degrees
- moved SW1 229.6 mm to (93.2, 53.0)
- moved C1 225.8 mm to (84.8, 59.9), turned to 180 degrees
- moved R2 218.4 mm to (95.8, 64.6), turned to -90 degrees
- moved R1 216.9 mm to (90.8, 65.3), turned to 180 degrees
- moved P4 196.5 mm to (103.4, 61.7)
- moved C2 196.2 mm to (74.2, 66.2), turned to 90 degrees
- moved P3 196.1 mm to (103.4, 64.4)
- moved P5 152.4 mm to (18.4, 122.8), turned to 90 degrees
- moved R10 96.8 mm to (104.7, 119.2), turned to 180 degrees
- moved R11 83.4 mm to (90.2, 119.2)
- moved AMP1 76.3 mm to (-198.5, 21.0)
- moved AMP8 76.3 mm to (-196.6, 9.14)
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- renumbered R12 to R10, R10 to R12, TP3 to TP1, TP1 to TP3
Connections:
- net /Microcomputer/I2C SCL renamed /Microcomputer/I2C SCL_1
- net /Microcomputer/I2C SDA renamed /Microcomputer/I2C SDA_1
- net /Microcomputer/TX_2 renamed /Microcomputer/I2C SCL_0
- C3 pad 1: /Microcomputer/3.3V -> /Microcomputer/5V
- C4 pad 1: /Microcomputer/5V -> /Microcomputer/3.3V
- C5 pad 1: /Microcomputer/3.3V -> /Microcomputer/5V
- C6 pad 1: /Microcomputer/5V -> /Microcomputer/3.3V
- C7 pad 1: /Microcomputer/5V -> /Microcomputer/3.3V
- J1 pad 1: Earth -> /Power/IN+
- J1 pad 2: /Power/IN+ -> Earth
- P1 pad 1: /Microcomputer/5V -> /Microcomputer/3.3V
- P1 pad 10: /Microcontroller/SPI_CS -> /Microcontroller/TX_1
- P1 pad 11: /Microcontroller/SPI_DC -> /Microcontroller/RX_1
- P1 pad 17: /Microcontroller/SPI_MOSI -> unconnected-(P1-Pin_17-Pad17)
- P1 pad 18: /Microcontroller/SPI_SCK -> unconnected-(P1-Pin_18-Pad18)
- P1 pad 19: /Microcontroller/SPI_MISO -> unconnected-(P1-Pin_19-Pad19)
- P1 pad 2: /Microcomputer/5V -> /Microcomputer/3.3V
- P1 pad 21: /Microcomputer/3.3V -> /Microcomputer/5V
- P1 pad 24: /Microcomputer/3.3V -> /Microcomputer/5V
- P1 pad 26: /Microcontroller/SPI_MISO -> unconnected-(P1-Pin_26-Pad26)
- P1 pad 27: /Microcontroller/SPI_SCK -> unconnected-(P1-Pin_27-Pad27)
- P1 pad 28: /Microcontroller/SPI_MOSI -> unconnected-(P1-Pin_28-Pad28)
- P1 pad 34: /Microcontroller/SPI_DC -> /Microcontroller/RX_1
- P1 pad 35: /Microcontroller/SPI_CS -> /Microcontroller/TX_1
- P1 pad 43: /Microcomputer/5V -> /Microcomputer/3.3V
- P1 pad 44: /Microcomputer/5V -> /Microcomputer/3.3V
- P3 pad 1: /Microcomputer/5V -> /Microcomputer/3.3V
- P3 pad 10: unconnected-(P3-Pin_10-Pad10) -> /Microcomputer/SPI MOSI
- P3 pad 11: unconnected-(P3-Pin_11-Pad11) -> /Microcomputer/SPI MISO
- P3 pad 12: unconnected-(P3-Pin_12-Pad12) -> /Microcomputer/SPI CLK
- P3 pad 6: unconnected-(P3-Pin_6-Pad6) -> /Microcomputer/TX_5
- P3 pad 7: unconnected-(P3-Pin_7-Pad7) -> /Microcomputer/RX_5
- P4 pad 1: /Microcomputer/TX_0 -> /Microcomputer/5V
- P4 pad 2: /Microcomputer/RX_0 -> /Microcomputer/5V
- P6 pad 1: /Microcontroller/SPI_DC -> /Microcomputer/SPI DC
- P6 pad 2: /Microcontroller/SPI_CS -> /Microcomputer/SPI CS
- P6 pad 3: /Microcontroller/SPI_SCK -> /Microcomputer/SPI CLK
- P6 pad 4: /Microcontroller/SPI_MISO -> /Microcomputer/SPI MISO
- P6 pad 5: /Microcontroller/SPI_MOSI -> /Microcomputer/SPI MOSI
- P6 pad 6: /Microcomputer/3.3V -> /Microcomputer/5V
- Q2 pad 2: /Microcomputer/3.3V -> /Microcomputer/5V
- R10 pad 2: /Signals Acquisition/Line C -> /Signals Acquisition/Line A
- R12 pad 2: /Signals Acquisition/Line A -> /Signals Acquisition/Line C
- R3 pad 2: /Microcomputer/3.3V -> /Microcomputer/5V
- R4 pad 1: /Microcomputer/3.3V -> /Microcomputer/5V
- R5 pad 2: /Microcomputer/5V -> /Microcomputer/3.3V
- R6 pad 1: /Microcomputer/5V -> /Microcomputer/3.3V
- TP1 pad 4: /Signals Acquisition/PT C-2 -> /Signals Acquisition/PT A-2
- TP3 pad 4: /Signals Acquisition/PT A-2 -> /Signals Acquisition/PT C-2
- U1 pad 2: /Microcomputer/3.3V -> /Microcomputer/5V
- U2 pad 1: /Microcomputer/RX_4 -> /Microcomputer/RX_3
- U2 pad 10: /Microcomputer/3.3V -> /Microcomputer/5V
- U2 pad 18: /Microcontroller/RX_0 -> /Microcontroller/RX_1
- U2 pad 19: /Microcomputer/5V -> /Microcomputer/3.3V
- U2 pad 2: /Microcomputer/3.3V -> /Microcomputer/5V
- U2 pad 20: /Microcontroller/TX_0 -> /Microcontroller/TX_1
- U2 pad 3: /Microcomputer/TX_4 -> /Microcomputer/TX_3
- U3 pad 4: /Microcomputer/5V -> /Microcomputer/3.3V
Routing:
- net (no net): track 427.3 -> 0.00 mm, vias 5 -> 0
- net Vref: track 206.7 -> 0.00 mm
- net Wave C: track 105.0 -> 0.00 mm
- net /Microcontroller/ADC1_6: track 71.5 -> 0.00 mm, vias 4 -> 0
- net Wave A: track 66.8 -> 0.00 mm
- net /Microcontroller/ADC1_3: track 63.7 -> 0.00 mm, vias 1 -> 0
- net /Microcontroller/ADC1_4: track 60.1 -> 0.00 mm
- net /Microcontroller/ADC1_5: track 56.9 -> 0.00 mm, vias 1 -> 0
- net /Signals Conditioning/CT B-2: track 42.5 -> 0.00 mm, vias 12 -> 0
- net /Microcontroller/ADC1_1: track 36.9 -> 0.00 mm, vias 1 -> 0
- net Net-(Q1-C): track 0.00 -> 35.4 mm
- net Net-(AMP3B-+): track 35.3 -> 0.00 mm, vias 1 -> 0
- net Net-(AMP2B--): track 29.1 -> 0.00 mm, vias 2 -> 0
- net Net-(AMP8A--): track 28.0 -> 0.00 mm, vias 2 -> 0
- net Earth: track 37.2 -> 9.77 mm, vias 26 -> 4
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