File: boards/v5.0/Microcomputer.kicad_sch (KiCad schematic)
At the start: 3 parts, among them P3 Pin Socket 2.54mm 2x20

Commit message: Update board v5.0 docs
Parts:
- P3: footprint (none) -> Connector_PinSocket_2.54mm:PinSocket_2x20_P2.54mm_Vertical
Changed lines of the file:
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@@
       (effects (font (size 1.27 1.27)) hide)
     )
-    (property "Footprint" "" (at 88.9 105.41 0)
+    (property "Footprint" "Connector_PinSocket_2.54mm:PinSocket_2x20_P2.54mm_Vertical" (at 88.9 105.41 0)
       (effects (font (size 1.27 1.27)) hide)
     )

Commit message: Update in the V5 board
Parts:
- removed P3: Pin Socket 2.54mm 2x20, Connector_PinSocket_2.54mm:PinSocket_2x20_P2.54mm_Vertical, symbol Connector_Generic:Conn_02x20_Counter_Clockwise
- added P4, P5: Conn_01x20, Connector_PinHeader_2.54mm:PinHeader_1x20_P2.54mm_Vertical, symbol Connector_Generic:Conn_01x20
Connections:
- net 3.3V: now also C7.1, P4.1 (Pin_1), P4.9 (Pin_9)
- net 5V: now also P5.1 (Pin_1), P5.2 (Pin_2); no longer C7.1
- net Earth: now also P4.13 (Pin_13), P4.20 (Pin_20), P4.5 (Pin_5), P5.10 (Pin_10), P5.15 (Pin_15), P5.17 (Pin_17), P5.3 (Pin_3), P5.7 (Pin_7)
- net RX_0: now also P5.5 (Pin_5)
- net RX_3: now also P4.14 (Pin_14)
- net RX_4: now also P5.8 (Pin_8)
- net TX_0: now also P5.4 (Pin_4)
- net TX_3: now also P5.14 (Pin_14)
- net TX_4: now also P4.4 (Pin_4)
- new net I2C SCL_0: P4.8 (Pin_8)
- new net I2C SCL_1: P4.3 (Pin_3)
- new net I2C SDA_0: P5.11 (Pin_11)
- new net I2C SDA_1: P4.2 (Pin_2)
- new net RX_5: P4.7 (Pin_7)
- new net SPI CLK: P4.12 (Pin_12)
- new net SPI CS: P5.12 (Pin_12)
- new net SPI DC: P5.13 (Pin_13)
- new net SPI MISO: P4.11 (Pin_11)
- new net SPI MOSI: P4.10 (Pin_10)
- new net TX_5: P4.6 (Pin_6)
Other:
- note removed: "-55 to +125"
- note removed: "0 to +70"
- note removed: "2 to 3"
- note removed: "5"
- note removed: "A"
- note removed: "Capacitor Operation Temperature"
- note removed: "Input Voltage - Vin"
- note removed: "Nominal Current Range"
- note removed: "Operating Temperature Range"
- note removed: "Orange Pi Zero 2W Operation Temperature"
- note removed: "Rating"
- note removed: "Specifications"
- note removed: "Unit"
- note removed: "Value"
- note removed: "Vdc"
- note removed: "°C"
- moved on the sheet: C7, C8
