File: boards/v5.0/Microcontroller.kicad_sch (KiCad schematic)
At the start: 10 parts, among them P1 Pin Socket 2.54mm 02x22, P2 Pin Socket 2.54mm 01x22, U2 TXS0108EPW

Commit message: Update board v5.0 docs
Parts:
- P1: footprint (none) -> Connector_PinSocket_2.54mm:PinSocket_2x22_P2.54mm_Vertical
- P2: footprint (none) -> Connector_PinSocket_2.54mm:PinSocket_1x22_P2.54mm_Vertical
Other:
- note added: "0.4"
- note removed: "0.5"
- company: Power Vision -> Lucas Rayan Guerra da Silva
- moved on the sheet: C4, C5, C6, P1, P2, R3, R4, R5, R6, U2

Commit message: Update in the V5 board
Parts:
- removed P1: Pin Socket 2.54mm 02x22, Connector_PinSocket_2.54mm:PinSocket_2x22_P2.54mm_Vertical, symbol Connector_Generic:Conn_02x22_Counter_Clockwise
- added P1, P2: Pin Socket 2.54mm 01x22, Connector_PinSocket_2.54mm:PinSocket_1x22_P2.54mm_Vertical, symbol Connector_Generic:Conn_01x22
- renumbered P2 to P3
Connections:
- net 3.3V: now also P1.1 (Pin_1), P1.2 (Pin_2), P2.1 (Pin_1), P2.2 (Pin_2)
- net ADC1_2: now also P1.13 (Pin_13)
- net ADC1_3: now also P1.4 (Pin_4), P2.13 (Pin_13)
- net ADC1_4: now also P1.5 (Pin_5)
- net ADC1_5: now also P1.6 (Pin_6)
- net ADC1_6: now also P1.7 (Pin_7)
- net Earth: now also P1.22 (Pin_22), P2.22 (Pin_22)
- net GPIO_17: now also P1.8 (Pin_8)
- net I2C_SCL: now also P1.15 (Pin_15), P2.15 (Pin_15)
- net I2C_SDA: now also P1.12 (Pin_12), P2.12 (Pin_12)
- net RESET: now also P1.3 (Pin_3), P2.3 (Pin_3)
- net RX_0: no longer U2.18 (B2)
- net TX_0: no longer U2.20 (B1)
- net Vin: now also P1.21 (Pin_21), P2.21 (Pin_21)
- new net RX_1: P1.11 (Pin_11), P2.11 (Pin_11), U2.18 (B2)
- new net TX_1: P1.10 (Pin_10), P2.10 (Pin_10), U2.20 (B1)
Other:
- note removed: "-40 to +65"
- note removed: "-40 to +85"
- note removed: "-55 to +125"
- note removed: "0.4"
- note removed: "5"
- note removed: "A"
- note removed: "Capacitor Operation Temperature"
- note removed: "ESP32-S3 Operation Temperature"
- note removed: "Input Voltage - Vin"
- note removed: "Nominal Current"
- note removed: "Operating Temperature Range"
- note removed: "Rating"
- note removed: "Specifications"
- note removed: "TXS0108E Operation Temperature"
- note removed: "Unit"
- note removed: "Value"
- note removed: "Vdc"
- note removed: "°C"

Commit message: Add Jupyter notebook for calculating possible sample rates
- Introduced a new notebook `possible_sample_rates.ipynb` that calculates sample rates based on a base frequency of 60Hz.
- The notebook iterates through a range of values to compute and print sample rates, frequencies, microseconds, and remainders for specific conditions.
Parts:
- removed R3, R4, R5, R6: 1kΩ, Resistor_SMD:R_0603_1608Metric, symbol Device:R
Connections:
- net ADC1_2: now also P2.13 (Pin_13)
- net ADC1_3: no longer P2.13 (Pin_13)
- net GPIO_17: no longer names the net of P1.8 (Pin_8)
- net I2C SCL: no longer names the net of U2.9 (A8)
- net I2C SDA: no longer names the net of U2.8 (A7)
- net I2C_SCL renamed GPIO_9
- net GPIO_9: no longer U2.12 (B8)
- removed net I2C_SDA: P1.12 (Pin_12), P2.12 (Pin_12), U2.13 (B7)
