File: boards/v5.0/Power.kicad_sch (KiCad schematic)
At the start: 9 parts, among them Q1 FZT948TA, Q2 FZT948TA, SW1 SS-12D00G 4mm, U1 LD1086#50

Commit message: Update in the V5 board
Other:
- note removed: "-55 to +125"
- note removed: "-55 to +150"
- note removed: "-65 to +150"
- note removed: "14"
- note removed: "30"
- note removed: "4"
- note removed: "5"
- note removed: "6"
- note removed: "A"
- note removed: "Capacitor Operation Temperature"
- note removed: "FZT948TA Operation Temperature"
- note removed: "LD1086 Operation Temperature"
- note removed: "Maximum Input Voltage"
- note removed: "Minimum Input Voltage"
- note removed: "Nominal Current"
- note removed: "Operating Temperature Range"
- note removed: "Output Voltage"
- note removed: "Rating"
- note removed: "Short circuit current"
- note removed: "Specifications"
- note removed: "Unit"
- note removed: "Value"
- note removed: "Vdc"
- note removed: "°C"
- title: Power -> Power Schematic
